Commit message: Update urdf to traxxas rally car

File: f1tenth_description/urdf/traxxas_rally.urdf.xacro (robot description, xacro)
@@ -1,6 +1,7 @@
 <?xml version="1.0"?>
-<!-- em_3905.urdf.xacro
-This file defines a model of a Traxxas(R) E-Maxx(R) #3905 RC (Radio Controlled)
-truck.
+<!-- traxxas_rally.urdf.xacro
+This file defines a model of a Traxxas Ford Fiesta ST Rally RTR 1/10 Rally Car.
+The exact specifications and dimensiosn are found here:
+https://www.hobbytown.com/traxxas-ford-fiesta-st-rally-rtr-1-10-4wd-rally-car-tra74054-4-r5/p696016
 Lengths are measured in meters, angles are measured in radians, and masses are
 measured in kilograms. All of these values are approximations.
@@ -33,6 +34,6 @@
   <!-- chassis_length is measured along the x axis, chassis_width
        along the y axis, and chassis_height along the z axis. -->
-  <xacro:property name="chassis_length" value="0.258"/>
-  <xacro:property name="chassis_width" value="0.168"/>
+  <xacro:property name="chassis_length" value="0.535"/>
+  <xacro:property name="chassis_width" value="0.281"/>
   <xacro:property name="chassis_height" value="0.01"/>
   <xacro:property name="chassis_mass" value="2.788"/>
@@ -56,6 +57,6 @@
   <xacro:property name="hub_dia" value="0.09652"/>
   <xacro:property name="tire_dia" value="0.14605"/>
-  <xacro:property name="tire_width" value="0.0889"/>
-  <xacro:property name="hex_hub_depth" value="0.01445"/>
+  <xacro:property name="tire_width" value="0.0444"/>
+  <xacro:property name="hex_hub_depth" value="0.0022"/>
   <xacro:property name="wheel_mass" value="0.29"/>
   <!-- hex_hub_dist is the distance between left and right hex hubs when
@@ -63,7 +64,7 @@
        from a U joint to the corresponding hex hub. wheel_travel is the
        vertical wheel travel. -->
-  <xacro:property name="wheelbase" value="0.335"/>
+  <xacro:property name="wheelbase" value="0.324"/>
   <xacro:property name="hex_hub_dist" value="0.365"/>
-  <xacro:property name="axle_length" value="0.03"/>
+  <xacro:property name="axle_length" value="0.02"/>
   <xacro:property name="wheel_travel" value="0.084"/>
   <xacro:property name="shock_z_offset" value="0.0655"/>
@@ -199,10 +200,10 @@
       <type>transmission_interface/SimpleTransmission</type>
       <joint name="${lr_prefix}_${fr_prefix}_shock">
-        <hardwareInterface>EffortJointInterface</hardwareInterface>
+        <hardwareInterface>hardware_interface/EffortJointInterface</hardwareInterface>
       </joint>
       <actuator name="${lr_prefix}_${fr_prefix}_shock_act">
         <!-- This hardwareInterface element exists for compatibility
              with ROS Hydro. -->
-        <hardwareInterface>EffortJointInterface</hardwareInterface>
+        <hardwareInterface>hardware_interface/EffortJointInterface</hardwareInterface>
         <mechanicalReduction>1</mechanicalReduction>
       </actuator>
@@ -226,10 +227,10 @@
       <type>transmission_interface/SimpleTransmission</type>
       <joint name="${lr_prefix}_${fr_prefix}_axle">
-        <hardwareInterface>EffortJointInterface</hardwareInterface>
+        <hardwareInterface>hardware_interface/EffortJointInterface</hardwareInterface>
       </joint>
       <actuator name="${lr_prefix}_${fr_prefix}_axle_act">
         <!-- This hardwareInterface element exists for compatibility
              with ROS Hydro. -->
-        <hardwareInterface>EffortJointInterface</hardwareInterface>
+        <hardwareInterface>hardware_interface/EffortJointInterface</hardwareInterface>
         <mechanicalReduction>1</mechanicalReduction>
       </actuator>
@@ -282,10 +283,10 @@
       <type>transmission_interface/SimpleTransmission</type>
       <joint name="${lr_prefix}_steering_joint">
-        <hardwareInterface>EffortJointInterface</hardwareInterface>
+        <hardwareInterface>hardware_interface/EffortJointInterface</hardwareInterface>
       </joint>
       <actuator name="${lr_prefix}_steering_act">
         <!-- This hardwareInterface element exists for compatibility
              with ROS Hydro. -->
-        <hardwareInterface>EffortJointInterface</hardwareInterface>
+        <hardwareInterface>hardware_interface/EffortJointInterface</hardwareInterface>
         <mechanicalReduction>1</mechanicalReduction>
       </actuator>

Commit message: Add Intel RealSense Camera Plugin

File: f1tenth_description/urdf/traxxas_rally.urdf.xacro (robot description, xacro)
@@ -21,5 +21,5 @@
 you may not use this file except in compliance with the License.
 You may obtain a copy of the License at
-  http://www.apache.org/licenses/LICENSE-2.0
+http://www.apache.org/licenses/LICENSE-2.0
 Unless required by applicable law or agreed to in writing, software
 distributed under the License is distributed on an "AS IS" BASIS,
@@ -80,11 +80,11 @@
        num_pinion_gear_teeth = 19
        final_gear_ratio = (num_spur_gear_teeth / num_pinion_gear_teeth) *
-         5.22 = 18.68
+       5.22 = 18.68
        stall_torque = 0.549 N m
        axle_eff_limit = ((2 * stall_torque) * final_gear_ratio) / 4 =
-         5.12766 N m
+       5.12766 N m
        max_speed = 40 mph (30+ mph) = 17.8816 m/s
        axle_vel_limit = (2 * pi) * (max_speed / (pi * tire_dia)) =
-         244.8696 rad/s -->
+       244.8696 rad/s -->
   <xacro:property name="axle_eff_limit" value="5.12766"/>
   <xacro:property name="axle_vel_limit" value="244.8696"/>
@@ -114,13 +114,13 @@
        along the y axis, and height along the z axis. -->
   <xacro:macro name="solid_cuboid_inertial"
-               params="width depth height mass *origin">
+	       params="width depth height mass *origin">
     <inertial>
       <xacro:insert_block name="origin"/>
       <mass value="${mass}"/>
       <inertia ixx="${mass * (depth * depth + height * height) / 12}"
-               ixy="0" ixz="0"
-               iyy="${mass * (width * width + height * height) / 12}"
-               iyz="0"
-               izz="${mass * (width * width + depth * depth) / 12}"/>
+	       ixy="0" ixz="0"
+	       iyy="${mass * (width * width + height * height) / 12}"
+	       iyz="0"
+	       izz="${mass * (width * width + depth * depth) / 12}"/>
     </inertial>
   </xacro:macro>
@@ -129,15 +129,15 @@
        outer_rad are the tube's inner and outer radii, respectively. -->
   <xacro:macro name="thick_walled_tube_inertial"
-               params="inner_rad outer_rad height mass">
+	       params="inner_rad outer_rad height mass">
     <inertial>
       <mass value="${mass}"/>
       <inertia ixx="${(1 / 12) * mass * (3 * (inner_rad * inner_rad +
-                    outer_rad * outer_rad) + height * height)}"
-               ixy="0" ixz="0"
-               iyy="${(1 / 12) * mass * (3 * (inner_rad * inner_rad +
-                    outer_rad * outer_rad) + height * height)}"
-               iyz="0"
-               izz="${mass * (inner_rad * inner_rad +
-                    outer_rad * outer_rad) / 2}"/>
+		    outer_rad * outer_rad) + height * height)}"
+	       ixy="0" ixz="0"
+	       iyy="${(1 / 12) * mass * (3 * (inner_rad * inner_rad +
+		    outer_rad * outer_rad) + height * height)}"
+	       iyz="0"
+	       izz="${mass * (inner_rad * inner_rad +
+		    outer_rad * outer_rad) / 2}"/>
     </inertial>
   </xacro:macro>
@@ -148,7 +148,7 @@
       <child link="${prefix}_battery_offset"/>
       <origin xyz="${battery_x_offset - battery_length / 2}
-                   ${reflect * battery_dist / 2}
-                   0"
-              rpy="${reflect * battery_comp_angle} 0 0"/>
+		   ${reflect * battery_dist / 2}
+		   0"
+	      rpy="${reflect * battery_comp_angle} 0 0"/>
     </joint>
     <link name="${prefix}_battery_offset">
@@ -159,23 +159,23 @@
       <child link="${prefix}_battery"/>
       <origin xyz="0
-                   ${reflect * battery_width / 2}
-                   ${(battery_height / 2) - battery_comp_depth}"/>
+		   ${reflect * battery_width / 2}
+		   ${(battery_height / 2) - battery_comp_depth}"/>
     </joint>
     <link name="${prefix}_battery">
       <visual>
-        <geometry>
-          <box size="${battery_length} ${battery_width} ${battery_height}"/>
-        </geometry>
-        <material name="battery_mat"/>
+	<geometry>
+	  <box size="${battery_length} ${battery_width} ${battery_height}"/>
+	</geometry>
+	<material name="battery_mat"/>
       </visual>
       <collision>
-        <geometry>
-          <box size="${battery_length} ${battery_width} ${battery_height}"/>
-        </geometry>
+	<geometry>
+	  <box size="${battery_length} ${battery_width} ${battery_height}"/>
+	</geometry>
       </collision>
       <xacro:solid_cuboid_inertial
-         width="${battery_length}" depth="${battery_width}"
-         height="${battery_height}" mass="${battery_mass}">
-        <origin/>
+	  width="${battery_length}" depth="${battery_width}"
+	  height="${battery_height}" mass="${battery_mass}">
+	<origin/>
       </xacro:solid_cuboid_inertial>
     </link>
@@ -186,25 +186,25 @@
   <!-- Shock absorber -->
   <xacro:macro name="shock"
-               params="lr_prefix fr_prefix lr_reflect fr_reflect child">
+	       params="lr_prefix fr_prefix lr_reflect fr_reflect child">
     <joint name="${lr_prefix}_${fr_prefix}_shock" type="prismatic">
       <parent link="chassis"/>
       <child link="${child}"/>
       <origin xyz="${fr_reflect * wheelbase / 2}
-                   ${lr_reflect * ((hex_hub_dist / 2) - axle_length)}
-                   ${(wheel_travel / 2) - shock_z_offset}"/>
+		   ${lr_reflect * ((hex_hub_dist / 2) - axle_length)}
+		   ${(wheel_travel / 2) - shock_z_offset}"/>
       <axis xyz="0 0 -1"/>
       <limit lower="${-wheel_travel / 2}" upper="${wheel_travel / 2}"
-             effort="${shock_eff_limit}" velocity="${shock_vel_limit}"/>
+	     effort="${shock_eff_limit}" velocity="${shock_vel_limit}"/>
     </joint>
     <transmission name="${lr_prefix}_${fr_prefix}_shock_trans">
       <type>transmission_interface/SimpleTransmission</type>
       <joint name="${lr_prefix}_${fr_prefix}_shock">
-        <hardwareInterface>hardware_interface/EffortJointInterface</hardwareInterface>
+	<hardwareInterface>hardware_interface/EffortJointInterface</hardwareInterface>
       </joint>
       <actuator name="${lr_prefix}_${fr_prefix}_shock_act">
-        <!-- This hardwareInterface element exists for compatibility
-             with ROS Hydro. -->
-        <hardwareInterface>hardware_interface/EffortJointInterface</hardwareInterface>
-        <mechanicalReduction>1</mechanicalReduction>
+	<!-- This hardwareInterface element exists for compatibility
+	     with ROS Hydro. -->
+	<hardwareInterface>hardware_interface/EffortJointInterface</hardwareInterface>
+	<mechanicalReduction>1</mechanicalReduction>
       </actuator>
     </transmission>
@@ -216,5 +216,5 @@
     </link>
     <!-- The left and right axles have the same axis so that identical
-         rotation values cause the wheels to rotate in the same direction. -->
+	 rotation values cause the wheels to rotate in the same direction. -->
     <joint name="${lr_prefix}_${fr_prefix}_axle" type="continuous">
       <parent link="${lr_prefix}_${fr_prefix}_axle_carrier"/>
@@ -227,36 +227,36 @@
       <type>transmission_interface/SimpleTransmission</type>
       <joint name="${lr_prefix}_${fr_prefix}_axle">
-        <hardwareInterface>hardware_interface/EffortJointInterface</hardwareInterface>
+	<hardwareInterface>hardware_interface/EffortJointInterface</hardwareInterface>
       </joint>
       <actuator name="${lr_prefix}_${fr_prefix}_axle_act">
-        <!-- This hardwareInterface element exists for compatibility
-             with ROS Hydro. -->
-        <hardwareInterface>hardware_interface/EffortJointInterface</hardwareInterface>
-        <mechanicalReduction>1</mechanicalReduction>
+	<!-- This hardwareInterface element exists for compatibility
+	     with ROS Hydro. -->
+	<hardwareInterface>hardware_interface/EffortJointInterface</hardwareInterface>
+	<mechanicalReduction>1</mechanicalReduction>
       </actuator>
     </transmission>
     <link name="${lr_prefix}_${fr_prefix}_wheel">
       <visual>
-        <origin xyz="0
-                     ${lr_reflect * (axle_length - (tire_width /
-                     2 - hex_hub_depth))}
-                     0"/>
-        <geometry>
-          <cylinder radius="${tire_dia / 2}" length="${tire_width}"/>
-        </geometry>
-        <material name="tire_mat"/>
+	<origin xyz="0
+		     ${lr_reflect * (axle_length - (tire_width /
+		     2 - hex_hub_depth))}
+		     0"/>
+	<geometry>
+	  <cylinder radius="${tire_dia / 2}" length="${tire_width}"/>
+	</geometry>
+	<material name="tire_mat"/>
       </visual>
       <collision>
-        <origin xyz="0
-                     ${lr_reflect * (axle_length - (tire_width /
-                     2 - hex_hub_depth))}
-                     0"/>
-        <geometry>
-          <cylinder radius="${tire_dia / 2}" length="${tire_width}"/>
-        </geometry>
+	<origin xyz="0
+		     ${lr_reflect * (axle_length - (tire_width /
+		     2 - hex_hub_depth))}
+		     0"/>
+	<geometry>
+	  <cylinder radius="${tire_dia / 2}" length="${tire_width}"/>
+	</geometry>
       </collision>
       <xacro:thick_walled_tube_inertial
-          inner_rad="${hub_dia / 2}" outer_rad="${tire_dia / 2}"
-          height="${tire_width}" mass="${wheel_mass}"/>
+	  inner_rad="${hub_dia / 2}" outer_rad="${tire_dia / 2}"
+	  height="${tire_width}" mass="${wheel_mass}"/>
     </link>
     <gazebo reference="${lr_prefix}_${fr_prefix}_wheel">
@@ -266,8 +266,8 @@
   <!-- Front wheel -->
   <xacro:macro name="front_wheel"
-               params="lr_prefix fr_prefix lr_reflect fr_reflect">
+	       params="lr_prefix fr_prefix lr_reflect fr_reflect">
     <xacro:shock lr_prefix="${lr_prefix}" fr_prefix="${fr_prefix}"
-                 lr_reflect="${lr_reflect}" fr_reflect="${fr_reflect}"
-                 child="${lr_prefix}_steering_link"/>
+		 lr_reflect="${lr_reflect}" fr_reflect="${fr_reflect}"
+		 child="${lr_prefix}_steering_link"/>
     <link name="${lr_prefix}_steering_link">
       <xacro:null_inertial/>
@@ -278,29 +278,29 @@
       <axis xyz="0 0 1"/>
       <limit lower="${-degrees_45}" upper="${degrees_45}"
-             effort="${servo_stall_torque}" velocity="${servo_no_load_speed}"/>
+	     effort="${servo_stall_torque}" velocity="${servo_no_load_speed}"/>
     </joint>
     <transmission name="${lr_prefix}_steering_trans">
       <type>transmission_interface/SimpleTransmission</type>
       <joint name="${lr_prefix}_steering_joint">
-        <hardwareInterface>hardware_interface/EffortJointInterface</hardwareInterface>
+	<hardwareInterface>hardware_interface/EffortJointInterface</hardwareInterface>
       </joint>
       <actuator name="${lr_prefix}_steering_act">
-        <!-- This hardwareInterface element exists for compatibility
-             with ROS Hydro. -->
-        <hardwareInterface>hardware_interface/EffortJointInterface</hardwareInterface>
-        <mechanicalReduction>1</mechanicalReduction>
+	<!-- This hardwareInterface element exists for compatibility
+	     with ROS Hydro. -->
+	<hardwareInterface>hardware_interface/EffortJointInterface</hardwareInterface>
+	<mechanicalReduction>1</mechanicalReduction>
       </actuator>
     </transmission>
     <xacro:wheel lr_prefix="${lr_prefix}" fr_prefix="${fr_prefix}"
-                 lr_reflect="${lr_reflect}"/>
+		 lr_reflect="${lr_reflect}"/>
   </xacro:macro>
   <!-- Rear wheel -->
   <xacro:macro name="rear_wheel"
-               params="lr_prefix fr_prefix lr_reflect fr_reflect">
+	       params="lr_prefix fr_prefix lr_reflect fr_reflect">
     <xacro:shock lr_prefix="${lr_prefix}" fr_prefix="${fr_prefix}"
-                 lr_reflect="${lr_reflect}" fr_reflect="${fr_reflect}"
-                 child="${lr_prefix}_${fr_prefix}_axle_carrier"/>
+		 lr_reflect="${lr_reflect}" fr_reflect="${fr_reflect}"
+		 child="${lr_prefix}_${fr_prefix}_axle_carrier"/>
     <xacro:wheel lr_prefix="${lr_prefix}" fr_prefix="${fr_prefix}"
-                 lr_reflect="${lr_reflect}"/>
+		 lr_reflect="${lr_reflect}"/>
   </xacro:macro>
   <!-- base_link must have geometry so that its axes can be displayed in
@@ -309,5 +309,5 @@
     <visual>
       <geometry>
-        <box size="0.01 0.01 0.01"/>
+	<box size="0.01 0.01 0.01"/>
       </geometry>
       <material name="chassis_mat"/>
@@ -322,5 +322,5 @@
       <origin xyz="0 0 ${-chassis_height / 2}"/>
       <geometry>
-        <box size="${chassis_length} ${chassis_width} ${chassis_height}"/>
+	<box size="${chassis_length} ${chassis_width} ${chassis_height}"/>
       </geometry>
       <material name="chassis_mat"/>
@@ -329,10 +329,10 @@
       <origin xyz="0 0 ${-chassis_height / 2}"/>
       <geometry>
-        <box size="${chassis_length} ${chassis_width} ${chassis_height}"/>
+	<box size="${chassis_length} ${chassis_width} ${chassis_height}"/>
       </geometry>
     </collision>
     <xacro:solid_cuboid_inertial
-        width="${chassis_length}" depth="${chassis_width}"
-        height="${chassis_height}" mass="${chassis_mass}">
+	width="${chassis_length}" depth="${chassis_width}"
+	height="${chassis_height}" mass="${chassis_mass}">
       <origin xyz="0 0 ${-chassis_height / 2}"/>
     </xacro:solid_cuboid_inertial>
@@ -350,13 +350,20 @@
   <!-- Wheels -->
   <xacro:front_wheel lr_prefix="left" fr_prefix="front"
-                     lr_reflect="1" fr_reflect="1"/>
+		     lr_reflect="1" fr_reflect="1"/>
   <xacro:front_wheel lr_prefix="right" fr_prefix="front"
-                     lr_reflect="-1" fr_reflect="1"/>
+		     lr_reflect="-1" fr_reflect="1"/>
   <xacro:rear_wheel lr_prefix="left" fr_prefix="rear"
-                    lr_reflect="1" fr_reflect="-1"/>
+		    lr_reflect="1" fr_reflect="-1"/>
   <xacro:rear_wheel lr_prefix="right" fr_prefix="rear"
-                    lr_reflect="-1" fr_reflect="-1"/>
+		    lr_reflect="-1" fr_reflect="-1"/>
   <gazebo>
     <plugin name="gazebo_ros_control" filename="libgazebo_ros_control.so"/>
   </gazebo>
+  <!-- Sensors -->
+  <!-- Import macro for realsense-RS200 camera-->
+  <xacro:include filename="$(find realsense_gazebo_plugin)/urdf/realsense-RS200.macro.xacro"/>
+  <!-- Create camera instance -->
+  <xacro:realsense-rs200 prefix="" parent="chassis">
+    <origin xyz="0 0 0.1" rpy="0 0 0" />
+  </xacro:realsense-rs200>
 </robot>
