Commit message: Add car meshes and make them configurable

File: ucsd_f1tenth_description/urdf/sensors.xacro (robot description, xacro)
@@ -49,5 +49,5 @@
   <xacro:include filename="$(find realsense_gazebo_plugin)/urdf/realsense-RS200.macro.xacro"/>
   <xacro:realsense-rs200 prefix="" parent="chassis">
-    <origin xyz="0.15 0 0.15" rpy="0 0 0" />
+    <origin xyz="0.1 0 0.1" rpy="0 0 0" />
   </xacro:realsense-rs200>
 </robot>

File: ucsd_f1tenth_description/urdf/traxxas_rally.urdf.xacro (robot description, xacro)
@@ -29,4 +29,5 @@
 -->
 <robot name="em_3905" xmlns:xacro="http://www.ros.org/wiki/xacro">
+  <xacro:arg name="car_type" default="delorean" />
   <!-- Degree-to-radian conversions -->
   <xacro:property name="degrees_45" value="0.785398163"/>
@@ -36,5 +37,5 @@
   <xacro:property name="chassis_length" value="0.535"/>
   <xacro:property name="chassis_width" value="0.281"/>
-  <xacro:property name="chassis_height" value="0.01"/>
+  <xacro:property name="chassis_height" value="0.00"/>
   <xacro:property name="chassis_mass" value="2.788"/>
   <!-- battery_dist is the distance between the inner edges of the
@@ -320,12 +321,12 @@
   <link name="chassis">
     <visual>
-      <origin xyz="0 0 ${-chassis_height / 2}"/>
+      <origin xyz="0 0 ${-chassis_height}"/>
       <geometry>
-	<box size="${chassis_length} ${chassis_width} ${chassis_height}"/>
+        <mesh filename="package://ucsd_f1tenth_description/meshes/$(arg car_type).stl" />
       </geometry>
       <material name="chassis_mat"/>
     </visual>
     <collision>
-      <origin xyz="0 0 ${-chassis_height / 2}"/>
+      <origin xyz="0 0 ${-chassis_height}"/>
       <geometry>
 	<box size="${chassis_length} ${chassis_width} ${chassis_height}"/>
@@ -335,5 +336,5 @@
 	width="${chassis_length}" depth="${chassis_width}"
 	height="${chassis_height}" mass="${chassis_mass}">
-      <origin xyz="0 0 ${-chassis_height / 2}"/>
+      <origin xyz="0 0 ${-chassis_height}"/>
     </xacro:solid_cuboid_inertial>
   </link>
